Commit message: First Version Finished

File: bravo_cathode_protection/urdf/bravo_5_dynamics_pinocchio_cp.urdf (robot description, URDF)
Before this commit: robot bravo5, 10 links, 9 joints
Links:
- added link cp_probe_3
Joints:
- added joint cp_probe_3_joint: type fixed, parent cp_probe_1, child cp_probe_3, origin xyz=0 0 0 rpy=0 0 -1.57

Commit message: almost ready

File: bravo_cathode_protection/urdf/bravo_5_dynamics_pinocchio_cp.urdf (robot description, URDF)
Before this commit: robot bravo5, 11 links, 10 joints
Links:
- removed link world
Joints:
- removed joint base_static_joint
